File: sucker-one-ui-board.kicad_pcb (KiCad board)
At the start: 0 parts

Commit message: Finish v1.0 and create gerbers
Parts:
- added J1: 52271-1079, Molex-52271-1079-*:Molex-52271-1079-Manufacturer_Recommended, B.Cu at (81.7, 69.6)
- added Q1: BSS138, Package_TO_SOT_SMD:SOT-23, F.Cu at (70.0, 71.5)
- added R1: 10k, Resistor_SMD:R_0603_1608Metric, F.Cu at (77.9, 71.5)
- added R2: 10k, Resistor_SMD:R_0603_1608Metric, F.Cu at (77.9, 77.2)
- added SW1: LIFT, Button_Switch_SMD:SW_SPST_B3U-1000P, F.Cu at (73.7, 74.1)
- added SW2: LOW, Button_Switch_SMD:SW_SPST_B3U-1000P, F.Cu at (73.7, 86.6)
- added SW3: REVERSE, Button_Switch_SMD:SW_SPST_B3U-1000P, F.Cu at (73.7, 99.1)
- added SW4: TRIGGER, Button_Switch_SMD:SW_SPST_B3U-1000P, F.Cu at (90.2, 99.1)
- added SW5: DROP, Button_Switch_SMD:SW_SPST_B3U-1000P, F.Cu at (90.2, 74.1)
- added SW6: HIGH, Button_Switch_SMD:SW_SPST_B3U-1000P, F.Cu at (90.2, 86.6)
- added TP1: GND, TestPoint:TestPoint_Pad_D1.5mm, B.Cu at (81.0, 100.3)
- added TP10: 3v3, TestPoint:TestPoint_Pad_D1.5mm, B.Cu at (73.4, 100.3)
- added TP2: LIFT, TestPoint:TestPoint_Pad_D1.5mm, B.Cu at (81.0, 103.1)
- added TP3: LOW, TestPoint:TestPoint_Pad_D1.5mm, B.Cu at (88.6, 103.1)
- added TP4: DROP, TestPoint:TestPoint_Pad_D1.5mm, B.Cu at (83.6, 103.1)
- added TP5: REVERSE, TestPoint:TestPoint_Pad_D1.5mm, B.Cu at (91.2, 103.1)
- added TP6: HIGH, TestPoint:TestPoint_Pad_D1.5mm, B.Cu at (86.1, 103.1)
- added TP7: TRIGGER, TestPoint:TestPoint_Pad_D1.5mm, B.Cu at (93.7, 103.1)
- added TP8: LED DATA, TestPoint:TestPoint_Pad_D1.5mm, B.Cu at (96.3, 103.1)
- added TP9: +5V, TestPoint:TestPoint_Pad_D1.5mm, B.Cu at (78.5, 100.3)
- added U1: WS2812-2020, WS2812-2020:LED_WS2812-2020, F.Cu at (69.3, 75.1)
- added U10: WS2812-2020, WS2812-2020:LED_WS2812-2020, F.Cu at (94.6, 74.0)
- added U11: WS2812-2020, WS2812-2020:LED_WS2812-2020, F.Cu at (94.7, 86.5)
- added U12: WS2812-2020, WS2812-2020:LED_WS2812-2020, F.Cu at (94.6, 99.1)
- added U2: WS2812-2020, WS2812-2020:LED_WS2812-2020, F.Cu at (69.2, 86.7)
- added U3: WS2812-2020, WS2812-2020:LED_WS2812-2020, F.Cu at (69.2, 99.1)
- added U4: WS2812-2020, WS2812-2020:LED_WS2812-2020, F.Cu at (78.1, 74.1)
- added U5: WS2812-2020, WS2812-2020:LED_WS2812-2020, F.Cu at (78.1, 86.6)
- added U6: WS2812-2020, WS2812-2020:LED_WS2812-2020, F.Cu at (78.1, 99.2)
- added U7: WS2812-2020, WS2812-2020:LED_WS2812-2020, F.Cu at (85.9, 74.0)
- added U8: WS2812-2020, WS2812-2020:LED_WS2812-2020, F.Cu at (85.9, 86.6)
- added U9: WS2812-2020, WS2812-2020:LED_WS2812-2020, F.Cu at (85.9, 99.1)
Routing:
- net GND: track 0.00 -> 167.5 mm, vias 0 -> 6
- net +5V: track 0.00 -> 144.2 mm, vias 0 -> 13
- net +3V3: track 0.00 -> 98.4 mm, vias 0 -> 12
- net LED_DATA: track 0.00 -> 80.1 mm, vias 0 -> 2
- net REVERSE_BTN: track 0.00 -> 59.5 mm, vias 0 -> 4
- net DROP_BTN: track 0.00 -> 57.1 mm, vias 0 -> 8
- net LIFT_BTN: track 0.00 -> 55.6 mm, vias 0 -> 8
- net LOW_BTN: track 0.00 -> 52.5 mm, vias 0 -> 4
- net TRIGGER_BTN: track 0.00 -> 52.0 mm, vias 0 -> 6
- net HIGH_BTN: track 0.00 -> 44.2 mm, vias 0 -> 10
- net DO_DROP: track 0.00 -> 38.7 mm, vias 0 -> 6
- net DO_HIGH: track 0.00 -> 30.2 mm, vias 0 -> 4
- net Net-(U10-Pad3): track 0.00 -> 19.8 mm, vias 0 -> 2
- net Net-(J1-Pad9): track 0.00 -> 18.6 mm, vias 0 -> 4
- net DO_LIFT: track 0.00 -> 13.3 mm, vias 0 -> 2
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Other:
- board outline added: 36.4 x 48.3 mm
- copper layers 0 -> 2
- board text added: "+5V"
- board text added: "DROP"
- board text added: "GND"
- board text added: "HIGH"
- board text added: "LED DATA"
- board text added: "LIFT"
- board text added: "LOW"
- board text added: "REVERSE"
- board text added: "Sucker One UI Board v1.0"
- board text added: "TRIGGER"
