File: sucker-one-ui-board.kicad_sch (KiCad schematic)
At the start: 0 parts

Commit message: Finish v1.0 and create gerbers
Parts:
- added J1: 52271-1079, Molex-52271-1079-*:Molex-52271-1079-Manufacturer_Recommended, symbol MOLEX 10 Pin 1mm FFC con:52271-1079
- added Q1: BSS138, Package_TO_SOT_SMD:SOT-23, symbol Transistor_FET:BSS138
- added R1, R2: 10k, Resistor_SMD:R_0603_1608Metric, symbol Device:R
- added SW1: LIFT, Button_Switch_SMD:SW_SPST_B3U-1000P, symbol Switch:SW_SPST
- added SW2: LOW, Button_Switch_SMD:SW_SPST_B3U-1000P, symbol Switch:SW_SPST
- added SW3: REVERSE, Button_Switch_SMD:SW_SPST_B3U-1000P, symbol Switch:SW_SPST
- added SW4: TRIGGER, Button_Switch_SMD:SW_SPST_B3U-1000P, symbol Switch:SW_SPST
- added SW5: DROP, Button_Switch_SMD:SW_SPST_B3U-1000P, symbol Switch:SW_SPST
- added SW6: HIGH, Button_Switch_SMD:SW_SPST_B3U-1000P, symbol Switch:SW_SPST
- added TP1: GND, TestPoint:TestPoint_Pad_D1.5mm, symbol Connector:TestPoint
- added TP10: 3v3, TestPoint:TestPoint_Pad_D1.5mm, symbol Connector:TestPoint
- added TP2: LIFT, TestPoint:TestPoint_Pad_D1.5mm, symbol Connector:TestPoint
- added TP3: LOW, TestPoint:TestPoint_Pad_D1.5mm, symbol Connector:TestPoint
- added TP4: DROP, TestPoint:TestPoint_Pad_D1.5mm, symbol Connector:TestPoint
- added TP5: REVERSE, TestPoint:TestPoint_Pad_D1.5mm, symbol Connector:TestPoint
- added TP6: HIGH, TestPoint:TestPoint_Pad_D1.5mm, symbol Connector:TestPoint
- added TP7: TRIGGER, TestPoint:TestPoint_Pad_D1.5mm, symbol Connector:TestPoint
- added TP8: LED DATA, TestPoint:TestPoint_Pad_D1.5mm, symbol Connector:TestPoint
- added TP9: +5V, TestPoint:TestPoint_Pad_D1.5mm, symbol Connector:TestPoint
- added U1, U10, U11, U12, U2, U3, U4, U5, U6, U7, U8, U9: WS2812-2020, WS2812-2020:LED_WS2812-2020, symbol WS2812-2020:WS2812-2020
Connections:
- new net: U10.3 (DI), U7.1 (DO)
- new net: U11.3 (DI), U8.1 (DO)
- new net: J1.9, Q1.2 (S), R1.1
- new net: U1.1 (DO), U4.3 (DI)
- new net: U2.1 (DO), U5.3 (DI)
- new net: U12.3 (DI), U9.1 (DO)
- new net: U3.1 (DO), U6.3 (DI)
- new net +3V3: J1.2, Q1.1 (G), R1.2, SW1.2 (B), SW2.2 (B), SW3.2 (B), SW4.2 (B), SW5.2 (B), SW6.2 (B), TP10.1
- new net +5V: J1.1, R2.2, TP9.1, U1.4 (VDD), U10.4 (VDD), U11.4 (VDD), U12.4 (VDD), U2.4 (VDD), U3.4 (VDD), U4.4 (VDD), U5.4 (VDD), U6.4 (VDD), U7.4 (VDD), U8.4 (VDD), U9.4 (VDD)
- new net DO_DROP: U10.1 (DO), U2.3 (DI)
- new net DO_HIGH: U11.1 (DO), U3.3 (DI)
- new net DO_LIFT: U4.1 (DO), U7.3 (DI)
- new net DO_LOW: U5.1 (DO), U8.3 (DI)
- new net DO_REV: U6.1 (DO), U9.3 (DI)
- new net DROP_BTN: J1.4, SW5.1 (A), TP4.1
- new net GND: J1.10, J1.MP1, J1.MP2, TP1.1, U1.2 (GND), U10.2 (GND), U11.2 (GND), U12.2 (GND), U2.2 (GND), U3.2 (GND), U4.2 (GND), U5.2 (GND), U6.2 (GND), U7.2 (GND), U8.2 (GND), U9.2 (GND)
- new net HIGH_BTN: J1.6, SW6.1 (A), TP6.1
- new net LED_DATA: Q1.3 (D), R2.1, TP8.1, U1.3 (DI)
- new net LIFT_BTN: J1.3, SW1.1 (A), TP2.1
- new net LOW_BTN: J1.5, SW2.1 (A), TP3.1
- new net REVERSE_BTN: J1.7, SW3.1 (A), TP5.1
- new net TRIGGER_BTN: J1.8, SW4.1 (A), TP7.1
- no-connect marks 0 -> 1
Other:
- note added: "3v3 <> 5v Logic Level Shift"
