File: pixel-pump-ui-board.kicad_pcb (KiCad board)
At the start: 4 copper layers, 36.4 x 49.3 mm, 42 parts, among them J1 SM10B-SRSS-TB, SW1 B3U-1000P, SW2 B3U-1000P, SW3 B3U-1000P, SW4 B3U-1000P, SW5 B3U-1000P, SW6 B3U-1000P, U1 WS2812B-2020, U10 WS2812B-2020, U11 WS2812B-2020, U12 WS2812B-2020, U2 WS2812B-2020, U3 WS2812B-2020, U4 WS2812B-2020, U5 WS2812B-2020, U6 WS2812B-2020, U7 WS2812B-2020, U8 WS2812B-2020, U9 WS2812B-2020

Commit message: Add KiKit Tabs
Parts:
- added T1: Tab, kikit:Tab, F.Cu at (62.6, 75.0)
- added T2: Tab, kikit:Tab, F.Cu at (105.1, 75.0)
- added T3: Tab, kikit:Tab, F.Cu at (62.7, 100.0)
- added T4: Tab, kikit:Tab, F.Cu at (104.7, 100.0)
Changed lines of the file:
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@@
     )
+  )
+  (footprint "kikit:Tab" (layer "F.Cu")
+    (at 62.6364 75)
+    (descr "A symbol representing annotation for tab placement")
+    (property "Sheetfile" "pixel-pump-ui-board.kicad_sch")
+    (property "Sheetname" "")
+    (property "exclude_from_bom" "")
+    (attr exclude_from_pos_files exclude_from_bom)
+    (fp_text reference "T1" (at 0 -2) (layer "F.SilkS") hide
+      (effects (font (size 1 1) (thickness 0.15)))
+    )
+    (fp_text value "Tab" (at -2.75 -1) (layer "Dwgs.User")
+      (effects (font (size 1.2 1.2) (thickness 0.2)))
+    )
+    (fp_text user "KIKIT: width: 2.5mm" (at -5.5 0 90) (layer "Dwgs.User")
+      (effects (font (size 1 1) (thickness 0.15)))
+    )
+    (fp_line (start 0.25 0) (end -0.75 1) (layer "Dwgs.User") (width 0.3))
+    (fp_line (start 0.25 1) (end 0.25 -1) (layer "Dwgs.User") (width 0.3))
+    (fp_line (start 0.25 0) (end -2.75 0) (layer "Dwgs.User") (width 0.3))
+    (fp_line (start 0.25 0) (end -0.75 -1) (layer "Dwgs.User") (width 0.3))
+  )
+  (footprint "kikit:Tab" (layer "F.Cu")
+    (at 104.7316 100 180)
+    (descr "A symbol representing annotation for tab placement")
+    (property "Sheetfile" "pixel-pump-ui-board.kicad_sch")
+    (property "Sheetname" "")
+    (property "exclude_from_bom" "")
+    (attr exclude_from_pos_files exclude_from_bom)
+    (fp_text reference "T4" (at 0 -2) (layer "F.SilkS") hide
+      (effects (font (size 1 1) (thickness 0.15)))
+    )
+    (fp_text value "Tab" (at -2.75 -1) (layer "Dwgs.User")
+      (effects (font (size 1.2 1.2) (thickness 0.2)))
+    )
+    (fp_text user "KIKIT: width: 2.5mm" (at -5.5 0 90) (layer "Dwgs.User")
+      (effects (font (size 1 1) (thickness 0.15)))
+    )
+    (fp_line (start 0.25 1) (end 0.25 -1) (layer "Dwgs.User") (width 0.3))
+    (fp_line (start 0.25 0) (end -2.75 0) (layer "Dwgs.User") (width 0.3))
+    (fp_line (start 0.25 0) (end -0.75 -1) (layer "Dwgs.User") (width 0.3))
+    (fp_line (start 0.25 0) (end -0.75 1) (layer "Dwgs.User") (width 0.3))
   )
   (footprint "Fiducial:Fiducial_0.75mm_Mask1.5mm" (layer "F.Cu")
@@
     )
   )
+  (footprint "kikit:Tab" (layer "F.Cu")
+    (at 62.6618 100)
+    (descr "A symbol representing annotation for tab placement")
+    (property "Sheetfile" "pixel-pump-ui-board.kicad_sch")
+    (property "Sheetname" "")
+    (property "exclude_from_bom" "")
+    (attr exclude_from_pos_files exclude_from_bom)
+    (fp_text reference "T3" (at 0 -2) (layer "F.SilkS") hide
+      (effects (font (size 1 1) (thickness 0.15)))
+    )
+    (fp_text value "Tab" (at -2.75 -1) (layer "Dwgs.User")
+      (effects (font (size 1.2 1.2) (thickness 0.2)))
+    )
+    (fp_text user "KIKIT: width: 2.5mm" (at -5.5 0 90) (layer "Dwgs.User")
+      (effects (font (size 1 1) (thickness 0.15)))
+    )
+    (fp_line (start 0.25 0) (end -2.75 0) (layer "Dwgs.User") (width 0.3))
+    (fp_line (start 0.25 0) (end -0.75 -1) (layer "Dwgs.User") (width 0.3))
+    (fp_line (start 0.25 0) (end -0.75 1) (layer "Dwgs.User") (width 0.3))
+    (fp_line (start 0.25 1) (end 0.25 -1) (layer "Dwgs.User") (width 0.3))
+  )
   (footprint "Button_Switch_SMD:SW_SPST_B3U-1000P" (layer "F.Cu")
     (at 90.17 74.1426 90)
@@
     )
   )
+  (footprint "kikit:Tab" (layer "F.Cu")
+    (at 105.1126 75 180)
+    (descr "A symbol representing annotation for tab placement")
+    (property "Sheetfile" "pixel-pump-ui-board.kicad_sch")
+    (property "Sheetname" "")
+    (property "exclude_from_bom" "")
+    (attr exclude_from_pos_files exclude_from_bom)
+    (fp_text reference "T2" (at 0 -2) (layer "F.SilkS") hide
+      (effects (font (size 1 1) (thickness 0.15)))
+    )
+    (fp_text value "Tab" (at -2.75 -1) (layer "Dwgs.User")
+      (effects (font (size 1.2 1.2) (thickness 0.2)))
+    )
+    (fp_text user "KIKIT: width: 2.5mm" (at -5.5 0 90) (layer "Dwgs.User")
+      (effects (font (size 1 1) (thickness 0.15)))
+    )
+    (fp_line (start 0.25 0) (end -0.75 -1) (layer "Dwgs.User") (width 0.3))
+    (fp_line (start 0.25 0) (end -2.75 0) (layer "Dwgs.User") (width 0.3))
+    (fp_line (start 0.25 1) (end 0.25 -1) (layer "Dwgs.User") (width 0.3))
+    (fp_line (start 0.25 0) (end -0.75 1) (layer "Dwgs.User") (width 0.3))
+  )
   (footprint "kibuzzard-6108471A" (layer "B.Cu")

Commit message: Panelize
Parts:
- J1: footprint Connector_JST:JST_SH_SM10B-SRSS-TB_1x10-1MP_P1.00mm_Horizontal -> SM10B-SRSS-TB:SM10B-SRSS-TB
- moved J1 0.46 mm to (81.6, 64.1)
Other:
- board text added: "REV 6"
- board text removed: "REV 5"
Changed lines of the file:
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@@
   (paper "A4")
   (title_block
-    (comment 4 "AISLER Project ID: JUGCKWAW")
+    (date "2023-02-24")
+    (rev "6")
   )
   (layers
@@
       (effects (font (size 1.2 1.2) (thickness 0.2)))
     )
-    (fp_text user "KIKIT: width: 2.5mm" (at -5.5 0 90) (layer "Dwgs.User")
+    (fp_text user "KIKIT: width: 2mm" (at -5.5 0 90) (layer "Dwgs.User")
       (effects (font (size 1 1) (thickness 0.15)))
     )
@@
       (effects (font (size 1.2 1.2) (thickness 0.2)))
     )
-    (fp_text user "KIKIT: width: 2.5mm" (at -5.5 0 90) (layer "Dwgs.User")
+    (fp_text user "KIKIT: width: 2mm" (at -5.5 0 90) (layer "Dwgs.User")
       (effects (font (size 1 1) (thickness 0.15)))
     )
@@
     )
   )
-  (footprint "Connector_JST:JST_SH_SM10B-SRSS-TB_1x10-1MP_P1.00mm_Horizontal" (layer "F.Cu")
-    (at 81.6356 64.516 180)
+  (footprint "SM10B-SRSS-TB:SM10B-SRSS-TB" (layer "F.Cu")
+    (at 81.6356 64.0588 180)
     (descr "JST SH series connector, SM10B-SRSS-TB (http://www.jst-mfg.com/product/pdf/eng/eSH.pdf), generated with kicad-footprint-generator")
     (tags "connector JST SH top entry")
@@
       (effects (font (size 1 1) (thickness 0.15)))
     )
-    (fp_text value "SM10B-SRSS-TB" (at 0 3.98) (layer "F.Fab")
+    (fp_text value "SM10B-SRSS-TB" (at 0 3.5228) (layer "F.Fab")
       (effects (font (size 1 1) (thickness 0.15)))
     )
-    (fp_text user "${REFERENCE}" (at 0 0) (layer "F.Fab")
+    (fp_text user "${REFERENCE}" (at 0 -0.4572) (layer "F.Fab")
       (effects (font (size 1 1) (thickness 0.15)))
     )
-    (fp_line (start 6.11 -1.785) (end 5.06 -1.785) (layer "F.SilkS") (width 0.12))
-    (fp_line (start 6.11 0.715) (end 6.11 -1.785) (layer "F.SilkS") (width 0.12))
-    (fp_line (start -6.11 0.715) (end -6.11 -1.785) (layer "F.SilkS") (width 0.12))
-    (fp_line (start -5.06 -1.785) (end -5.06 -2.775) (layer "F.SilkS") (width 0.12))
-    (fp_line (start -6.11 -1.785) (end -5.06 -1.785) (layer "F.SilkS") (width 0.12))
-    (fp_line (start -4.94 2.685) (end 4.94 2.685) (layer "F.SilkS") (width 0.12))
-    (fp_line (start -6.9 -3.28) (end -6.9 3.28) (layer "F.CrtYd") (width 0.05))
-    (fp_line (start 6.9 3.28) (end 6.9 -3.28) (layer "F.CrtYd") (width 0.05))
-    (fp_line (start 6.9 -3.28) (end -6.9 -3.28) (layer "F.CrtYd") (width 0.05))
-    (fp_line (start -6.9 3.28) (end 6.9 3.28) (layer "F.CrtYd") (width 0.05))
-    (fp_line (start -6 2.575) (end 6 2.575) (layer "F.Fab") (width 0.1))
-    (fp_line (start -5 -1.675) (end -4.5 -0.967893) (layer "F.Fab") (width 0.1))
-    (fp_line (start -6 -1.675) (end 6 -1.675) (layer "F.Fab") (width 0.1))
-    (fp_line (start 6 -1.675) (end 6 2.575) (layer "F.Fab") (width 0.1))
-    (fp_line (start -6 -1.675) (end -6 2.575) (layer "F.Fab") (width 0.1))
-    (fp_line (start -4.5 -0.967893) (end -4 -1.675) (layer "F.Fab") (width 0.1))
-    (pad "1" smd roundrect (at -4.5 -2 180) (size 0.6 1.55) (layers "F.Cu" "F.Paste" "F.Mask") (roundrect_rratio 0.25)
+    (fp_line (start 6.11 0.2578) (end 6.11 -2.2422) (layer "F.SilkS") (width 0.12))
+    (fp_line (start 6.11 -2.2422) (end 5.06 -2.2422) (layer "F.SilkS") (width 0.12))
+    (fp_line (start -4.94 2.2278) (end 4.94 2.2278) (layer "F.SilkS") (width 0.12))
+    (fp_line (start -6.11 0.2578) (end -6.11 -2.2422) (layer "F.SilkS") (width 0.12))
+    (fp_line (start -6.11 -2.2422) (end -5.06 -2.2422) (layer "F.SilkS") (width 0.12))
+    (fp_line (start -5.06 -2.2422) (end -5.06 -3.2322) (layer "F.SilkS") (width 0.12))
+    (fp_line (start 6.9 2.8228) (end 6.9 -3.7372) (layer "F.CrtYd") (width 0.05))
+    (fp_line (start 6.9 -3.7372) (end -6.9 -3.7372) (layer "F.CrtYd") (width 0.05))
+    (fp_line (start -6.9 -3.7372) (end -6.9 2.8228) (layer "F.CrtYd") (width 0.05))
+    (fp_line (start -6.9 2.8228) (end 6.9 2.8228) (layer "F.CrtYd") (width 0.05))
+    (fp_line (start -6 -2.1322) (end -6 2.1178) (layer "F.Fab") (width 0.1))
+    (fp_line (start -5 -2.1322) (end -4.5 -1.425093) (layer "F.Fab") (width 0.1))
+    (fp_line (start -4.5 -1.425093) (end -4 -2.1322) (layer "F.Fab") (width 0.1))
+    (fp_line (start -6 2.1178) (end 6 2.1178) (layer "F.Fab") (width 0.1))
+    (fp_line (start -6 -2.1322) (end 6 -2.1322) (layer "F.Fab") (width 0.1))
+    (fp_line (start 6 -2.1322) (end 6 2.1178) (layer "F.Fab") (width 0.1))
+    (pad "1" smd roundrect (at -4.5 -2.4572 180) (size 0.6 1.55) (layers "F.Cu" "F.Paste" "F.Mask") (roundrect_rratio 0.25)
       (net 1 "GND") (pinfunction "Pin_1") (pintype "passive"))
-    (pad "2" smd roundrect (at -3.5 -2 180) (size 0.6 1.55) (layers "F.Cu" "F.Paste" "F.Mask") (roundrect_rratio 0.25)
+    (pad "2" smd roundrect (at -3.5 -2.4572 180) (size 0.6 1.55) (layers "F.Cu" "F.Paste" "F.Mask") (roundrect_rratio 0.25)
       (net 9 "LED_DATA") (pinfunction "Pin_2") (pintype "passive"))
-    (pad "3" smd roundrect (at -2.5 -2 180) (size 0.6 1.55) (layers "F.Cu" "F.Paste" "F.Mask") (roundrect_rratio 0.25)
+    (pad "3" smd roundrect (at -2.5 -2.4572 180) (size 0.6 1.55) (layers "F.Cu" "F.Paste" "F.Mask") (roundrect_rratio 0.25)
       (net 7 "TRIGGER_BTN") (pinfunction "Pin_3") (pintype "passive"))
-    (pad "4" smd roundrect (at -1.5 -2 180) (size 0.6 1.55) (layers "F.Cu" "F.Paste" "F.Mask") (roundrect_rratio 0.25)
+    (pad "4" smd roundrect (at -1.5 -2.4572 180) (size 0.6 1.55) (layers "F.Cu" "F.Paste" "F.Mask") (roundrect_rratio 0.25)
       (net 4 "REVERSE_BTN") (pinfunction "Pin_4") (pintype "passive"))
-    (pad "5" smd roundrect (at -0.5 -2 180) (size 0.6 1.55) (layers "F.Cu" "F.Paste" "F.Mask") (roundrect_rratio 0.25)
+    (pad "5" smd roundrect (at -0.5 -2.4572 180) (size 0.6 1.55) (layers "F.Cu" "F.Paste" "F.Mask") (roundrect_rratio 0.25)
       (net 3 "HIGH_BTN") (pinfunction "Pin_5") (pintype "passive"))
-    (pad "6" smd roundrect (at 0.5 -2 180) (size 0.6 1.55) (layers "F.Cu" "F.Paste" "F.Mask") (roundrect_rratio 0.25)
+    (pad "6" smd roundrect (at 0.5 -2.4572 180) (size 0.6 1.55) (layers "F.Cu" "F.Paste" "F.Mask") (roundrect_rratio 0.25)
       (net 6 "LOW_BTN") (pinfunction "Pin_6") (pintype "passive"))
-    (pad "7" smd roundrect (at 1.5 -2 180) (size 0.6 1.55) (layers "F.Cu" "F.Paste" "F.Mask") (roundrect_rratio 0.25)
+    (pad "7" smd roundrect (at 1.5 -2.4572 180) (size 0.6 1.55) (layers "F.Cu" "F.Paste" "F.Mask") (roundrect_rratio 0.25)
       (net 5 "DROP_BTN") (pinfunction "Pin_7") (pintype "passive"))
-    (pad "8" smd roundrect (at 2.5 -2 180) (size 0.6 1.55) (layers "F.Cu" "F.Paste" "F.Mask") (roundrect_rratio 0.25)
+    (pad "8" smd roundrect (at 2.5 -2.4572 180) (size 0.6 1.55) (layers "F.Cu" "F.Paste" "F.Mask") (roundrect_rratio 0.25)
       (net 2 "LIFT_BTN") (pinfunction "Pin_8") (pintype "passive"))
-    (pad "9" smd roundrect (at 3.5 -2 180) (size 0.6 1.55) (layers "F.Cu" "F.Paste" "F.Mask") (roundrect_rratio 0.25)
+    (pad "9" smd roundrect (at 3.5 -2.4572 180) (size 0.6 1.55) (layers "F.Cu" "F.Paste" "F.Mask") (roundrect_rratio 0.25)
       (net 22 "+3V3") (pinfunction "Pin_9") (pintype "passive"))
-    (pad "10" smd roundrect (at 4.5 -2 180) (size 0.6 1.55) (layers "F.Cu" "F.Paste" "F.Mask") (roundrect_rratio 0.25)
+    (pad "10" smd roundrect (at 4.5 -2.4572 180) (size 0.6 1.55) (layers "F.Cu" "F.Paste" "F.Mask") (roundrect_rratio 0.25)
       (net 8 "+5V") (pinfunction "Pin_10") (pintype "passive"))
-    (pad "MP" smd roundrect (at 5.8 1.875 180) (size 1.2 1.8) (layers "F.Cu" "F.Paste" "F.Mask") (roundrect_rratio 0.2083333333)
+    (pad "MP" smd roundrect (at -5.8 1.4178 180) (size 1.2 1.8) (layers "F.Cu" "F.Paste" "F.Mask") (roundrect_rratio 0.2083333333)
       (net 1 "GND") (pinfunction "MountPin") (pintype "passive"))
-    (pad "MP" smd roundrect (at -5.8 1.875 180) (size 1.2 1.8) (layers "F.Cu" "F.Paste" "F.Mask") (roundrect_rratio 0.2083333333)
+    (pad "MP" smd roundrect (at 5.8 1.4178 180) (size 1.2 1.8) (layers "F.Cu" "F.Paste" "F.Mask") (roundrect_rratio 0.2083333333)
       (net 1 "GND") (pinfunction "MountPin") (pintype "passive"))
     (model "${KIPRJMOD}/components/SM10B-SRSS-TB/SM10B-SRSS-TB.STEP"
@@
       (effects (font (size 1.2 1.2) (thickness 0.2)))
     )
-    (fp_text user "KIKIT: width: 2.5mm" (at -5.5 0 90) (layer "Dwgs.User")
+    (fp_text user "KIKIT: width: 2mm" (at -5.5 0 90) (layer "Dwgs.User")
       (effects (font (size 1 1) (thickness 0.15)))
     )
@@
       (effects (font (size 1.2 1.2) (thickness 0.2)))
     )
-    (fp_text user "KIKIT: width: 2.5mm" (at -5.5 0 90) (layer "Dwgs.User")
+    (fp_text user "KIKIT: width: 2mm" (at -5.5 0 90) (layer "Dwgs.User")
       (effects (font (size 1 1) (thickness 0.15)))
     )
@@
   (gr_arc (start 86.62375 107.335437) (mid 87.759423 107.689128) (end 88.493376 108.625156) (layer "Edge.Cuts") (width 0.2))
   (gr_arc (start 74.856624 108.625156) (mid 71.723676 110.785439) (end 68.592437 108.62268) (layer "Edge.Cuts") (width 0.2))
-  (gr_text "REV 5" (at 81.6356 89.662) (layer "B.SilkS")
+  (gr_text "REV 6" (at 81.6356 89.662) (layer "B.SilkS")
     (effects (font (size 0.65 0.65) (thickness 0.13)) (justify mirror))
   )
